File: Hardware/Leiterplatte/Lixieuhr-Segment.brd (EAGLE design)
At the start: 40 x 60 mm, 17 parts, among them U1 APA102C, U10 APA102C, U2 APA102C, U3 APA102C, U4 APA102C, U5 APA102C, U6 APA102C, U7 APA102C, U8 APA102C, U9 APA102C

Commit message: Schaltpläne V02
Parts:
- removed FRAME1: HTL-A4-HA4H, 0_HTL_frame:HTL-A4-H
- removed JP2: (no value), jumper:JP4
- added C1, C10, C11, C12, C13, C14, C15, C16, C17, C18, C19, C2, C20, C3, C4, C5, C6, C7, C8, C9: 100nF, 0_HTL_MegaCard_V3:C0805
- added C21: (no value), rcl:E3,5-8
- added JP4: (no value), jumper:JP4
- added U11, U12, U13, U14, U15, U16, U17, U18, U19, U20: APA102C, APA102C:SON160P500X500X140-6N
Connections:
- new net N$23: U11.5, U12.2
- new net N$24: U12.5, U13.2
- new net N$25: U13.5, U14.2
- new net N$26: U14.5, U15.2
- new net N$27: U16.5, U17.2
- new net N$28: U17.5, U18.2
- new net N$29: U18.5, U19.2
- new net N$30: U19.5, U20.2
- new net N$31: U11.6, U12.1
- new net N$32: U12.6, U13.1
- new net N$33: U13.6, U14.1
- new net N$34: U14.6, U15.1
- new net N$36: U19.6, U20.1
- new net N$37: U16.6, U17.1
- new net N$38: U17.6, U18.1
- new net N$39: U18.6, U19.1
- new net N$43: JP4.2, U20.5
- new net N$44: JP4.3, U20.6
- new net N$47: U15.5, U16.2
- new net N$48: U15.6, U16.1
- net GND: now also C1.1, C10.1, C11.1, C12.1, C13.1, C14.1, C15.1, C16.1, C17.1, C18.1, C19.1, C2.1, C20.1, C21.-, C3.1, C4.1, C5.1, C6.1, C7.1, C8.1, C9.1, JP4.4, U11.3, U12.3, U13.3, U14.3, U15.3, U16.3, U17.3, U18.3, U19.3, U20.3; no longer JP2.4
- net N$21: now also U11.2; no longer JP2.2
- net N$22: now also U11.1; no longer JP2.3
- net V+: now also C1.2, C10.2, C11.2, C12.2, C13.2, C14.2, C15.2, C16.2, C17.2, C18.2, C19.2, C2.2, C20.2, C21.+, C3.2, C4.2, C5.2, C6.2, C7.2, C8.2, C9.2, JP4.1, U11.4, U12.4, U13.4, U14.4, U15.4, U16.4, U17.4, U18.4, U19.4, U20.4; no longer JP2.1
Routing:
- net N$46: track 8.42 -> 5.61 mm
- net N$19: track 8.63 -> 6.69 mm
- net N$22: track 41.8 -> 40.1 mm
- net V+: track 152.6 -> 151.0 mm
- net N$21: track 6.84 -> 5.81 mm

Commit message: Segmentplatine_V02
Parts:
- removed U$1, U$2, U$3, U$4: (no value), 0_HTL_holes:3,2
- C21: value (none) -> 1mF
- moved C21 315.9 mm to (22.6, 45.0)
- moved C20 284.9 mm to (32.8, 12.8), flipped to the bottom, turned to 180 degrees
- moved C19 273.7 mm to (26.0, 9.25), flipped to the bottom, turned to 180 degrees
- moved C18 265.7 mm to (19.2, 9.25), flipped to the bottom, turned to 180 degrees
- moved C16 262.1 mm to (12.5, 19.8), flipped to the bottom
- moved C17 260.7 mm to (12.5, 12.8), flipped to the bottom, turned to 180 degrees
- moved C13 257.9 mm to (32.8, 19.8), flipped to the bottom
- moved C15 257.3 mm to (19.2, 16.2), flipped to the bottom
- moved C14 256.0 mm to (26.0, 16.2), flipped to the bottom
- moved C12 252.6 mm to (26.0, 23.2), flipped to the bottom, turned to 180 degrees
- moved C10 250.0 mm to (32.8, 26.8), flipped to the bottom, turned to 180 degrees
- moved C11 244.4 mm to (19.2, 23.2), flipped to the bottom, turned to 180 degrees
- moved C8 235.8 mm to (12.5, 33.8), flipped to the bottom
- moved C9 234.5 mm to (12.5, 26.8), flipped to the bottom, turned to 180 degrees
- moved C4 234.5 mm to (32.8, 40.8), flipped to the bottom, turned to 180 degrees
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Routing:
- net GND: track 0.00 -> 102.2 mm, vias 0 -> 20
- net V+: track 151.0 -> 97.4 mm, vias 9 -> 19
- net N$22: track 40.1 -> 2.45 mm, vias 2 -> 0
- net N$17: track 30.4 -> 4.87 mm, vias 2 -> 0
- net N$7: track 27.6 -> 5.09 mm, vias 2 -> 0
- net N$3: track 25.7 -> 5.06 mm, vias 2 -> 0
- net N$44: track 0.00 -> 17.6 mm
- net N$8: track 26.9 -> 9.73 mm, vias 2 -> 0
- net N$43: track 0.00 -> 16.9 mm
- net N$18: track 22.6 -> 6.02 mm, vias 2 -> 0
- net N$2: track 17.7 -> 2.45 mm, vias 2 -> 0
- net N$32: track 0.00 -> 13.1 mm
- net N$11: track 13.0 -> 2.45 mm
- net N$12: track 15.2 -> 4.82 mm, vias 2 -> 0
- net N$4: track 18.9 -> 9.03 mm, vias 2 -> 0
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- added copper zone on layer 16, net V+
Other:
- board size 40 x 60 mm -> 45 x 50 mm
