File: Hardware/Leiterplatte/Master/Lixie_Master.brd (EAGLE design)
At the start: 20 x 43.6 mm, 9 parts, among them IC1 FT232RL, J1 65100516121, U1 ATTINY406-MFR

Commit message: Leiterplatten V05
Routing:
- net N$9: track 15.1 -> 12.9 mm
Other:
- outline, holes or cut-outs redrawn
Changed lines of the file:
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@@
 <setting verticaltext="up"/>
 </settings>
-<grid distance="25" unitdist="mil" unit="mil" style="lines" multiple="1" display="yes" altdistance="12.5" altunitdist="mil" altunit="mil"/>
+<grid distance="1" unitdist="mm" unit="mm" style="lines" multiple="1" display="yes" altdistance="12.5" altunitdist="mil" altunit="mil"/>
 <layers>
 <layer number="1" name="Top" color="4" fill="1" visible="yes" active="yes"/>
@@
 <wire x1="0" y1="0" x2="20" y2="0" width="0.4064" layer="20"/>
 <wire x1="20" y1="0" x2="20" y2="33.57" width="0.4064" layer="20"/>
-<wire x1="20" y1="33.57" x2="16" y2="33.57" width="0.4064" layer="20"/>
-<wire x1="4" y1="33.57" x2="0" y2="33.57" width="0.4064" layer="20"/>
+<wire x1="20" y1="33.57" x2="17" y2="33.57" width="0.4064" layer="20"/>
+<wire x1="3" y1="33.57" x2="0" y2="33.57" width="0.4064" layer="20"/>
 <wire x1="0" y1="33.57" x2="0" y2="0" width="0.4064" layer="20"/>
-<wire x1="4" y1="33.57" x2="4" y2="43.57" width="0.4064" layer="20"/>
-<wire x1="4" y1="43.57" x2="16" y2="43.57" width="0.4064" layer="20"/>
-<wire x1="16" y1="43.57" x2="16" y2="33.57" width="0.4064" layer="20"/>
+<wire x1="3" y1="33.57" x2="3" y2="43.57" width="0.4064" layer="20"/>
+<wire x1="3" y1="43.57" x2="17" y2="43.57" width="0.4064" layer="20"/>
+<wire x1="17" y1="43.57" x2="17" y2="33.57" width="0.4064" layer="20"/>
 </plain>
 <attributes>
@@
 <param name="mtCopper" value="0.035mm 0.035mm 0.035mm 0.035mm 0.035mm 0.035mm 0.035mm 0.035mm 0.035mm 0.035mm 0.035mm 0.035mm 0.035mm 0.035mm 0.035mm 0.035mm"/>
 <param name="mtIsolate" value="1.5mm 0.15mm 0.2mm 0.15mm 0.2mm 0.15mm 0.2mm 0.15mm 0.2mm 0.15mm 0.2mm 0.15mm 0.2mm 0.15mm 0.2mm"/>
-<param name="mdWireWire" value="8mil"/>
-<param name="mdWirePad" value="8mil"/>
-<param name="mdWireVia" value="8mil"/>
-<param name="mdPadPad" value="8mil"/>
-<param name="mdPadVia" value="8mil"/>
-<param name="mdViaVia" value="8mil"/>
-<param name="mdSmdPad" value="8mil"/>
-<param name="mdSmdVia" value="8mil"/>
-<param name="mdSmdSmd" value="8mil"/>
+<param name="mdWireWire" value="4mil"/>
+<param name="mdWirePad" value="4mil"/>
+<param name="mdWireVia" value="4mil"/>
+<param name="mdPadPad" value="4mil"/>
+<param name="mdPadVia" value="4mil"/>
+<param name="mdViaVia" value="4mil"/>
+<param name="mdSmdPad" value="4mil"/>
+<param name="mdSmdVia" value="4mil"/>
+<param name="mdSmdSmd" value="4mil"/>
 <param name="mdViaViaSameLayer" value="8mil"/>
 <param name="mnLayersViaInSmd" value="2"/>
-<param name="mdCopperDimension" value="40mil"/>
+<param name="mdCopperDimension" value="20mil"/>
 <param name="mdDrill" value="8mil"/>
 <param name="mdSmdStop" value="0mil"/>
-<param name="msWidth" value="10mil"/>
-<param name="msDrill" value="24mil"/>
+<param name="msWidth" value="5mil"/>
+<param name="msDrill" value="20mil"/>
 <param name="msMicroVia" value="9.99mm"/>
 <param name="msBlindViaRatio" value="0.5"/>
@@
 <contactref element="U1" pad="15"/>
 <contactref element="U$3" pad="2"/>
-<wire x1="11.45" y1="14.37" x2="11.9825" y2="14.37" width="0.254" layer="1"/>
-<wire x1="11.9825" y1="14.37" x2="12.3825" y2="13.97" width="0.254" layer="1"/>
-<via x="12.3825" y="13.97" extent="1-16" drill="0.5" shape="octagon"/>
-<wire x1="12.3825" y1="13.97" x2="12.3825" y2="10.16" width="0.254" layer="16"/>
-<via x="12.3825" y="10.16" extent="1-16" drill="0.5" shape="octagon"/>
-<wire x1="12.3825" y1="10.16" x2="15.67" y2="10.16" width="0.254" layer="1"/>
-<wire x1="15.67" y1="10.16" x2="17" y2="11.49" width="0.254" layer="1"/>
+<wire x1="17" y1="11.49" x2="16.062" y2="11.49" width="0.254" layer="1"/>
+<wire x1="16.062" y1="11.49" x2="14.732" y2="10.16" width="0.254" layer="1"/>
+<wire x1="14.732" y1="10.16" x2="12.954" y2="10.16" width="0.254" layer="1"/>
+<wire x1="12.954" y1="10.16" x2="12.7" y2="10.414" width="0.254" layer="1"/>
+<via x="12.7" y="10.414" extent="1-16" drill="0.6" shape="octagon"/>
+<wire x1="12.7" y1="10.414" x2="12.7" y2="14.224" width="0.254" layer="16"/>
+<wire x1="11.45" y1="14.37" x2="12.554" y2="14.37" width="0.254" layer="1"/>
+<wire x1="12.554" y1="14.37" x2="12.7" y2="14.224" width="0.254" layer="1"/>
+<via x="12.7" y="14.224" extent="1-16" drill="0.6" shape="octagon"/>
 </signal>
 <signal name="N$9">
 <contactref element="U1" pad="17"/>
 <contactref element="U$3" pad="3"/>
-<wire x1="10.4" y1="15.02" x2="10.4" y2="16.75" width="0.254" layer="1"/>
-<wire x1="10.4" y1="16.75" x2="10.795" y2="17.145" width="0.254" layer="1"/>
-<via x="10.795" y="17.145" extent="1-16" drill="0.5" shape="octagon"/>
-<wire x1="10.795" y1="17.145" x2="12.7" y2="17.145" width="0.254" layer="16"/>
-<wire x1="12.7" y1="17.145" x2="13.0175" y2="16.8275" width="0.254" layer="16"/>
-<wire x1="13.0175" y1="16.8275" x2="13.0175" y2="11.43" width="0.254" layer="16"/>
-<via x="13.0175" y="11.43" extent="1-16" drill="0.5" shape="octagon"/>
-<wire x1="13.0175" y1="11.43" x2="14.4" y2="11.43" width="0.254" layer="1"/>
-<wire x1="14.4" y1="11.43" x2="17" y2="14.03" width="0.254" layer="1"/>
+<wire x1="17" y1="14.03" x2="17" y2="13.571" width="0.254" layer="1"/>
+<wire x1="17" y1="13.571" x2="14.859" y2="11.43" width="0.254" layer="1"/>
+<wire x1="14.859" y1="11.43" x2="13.97" y2="11.43" width="0.254" layer="1"/>
+<wire x1="13.97" y1="11.43" x2="13.716" y2="11.684" width="0.254" layer="1"/>
+<via x="13.716" y="11.684" extent="1-16" drill="0.6" shape="octagon"/>
+<wire x1="13.716" y1="11.684" x2="13.716" y2="15.621" width="0.254" layer="16"/>
+<wire x1="13.716" y1="15.621" x2="13.335" y2="16.002" width="0.254" layer="16"/>
+<via x="13.335" y="16.002" extent="1-16" drill="0.6" shape="octagon"/>
+<wire x1="13.335" y1="16.002" x2="10.795" y2="16.002" width="0.254" layer="1"/>
+<wire x1="10.795" y1="16.002" x2="10.4" y2="15.607" width="0.254" layer="1"/>
+<wire x1="10.4" y1="15.02" x2="10.4" y2="15.607" width="0.254" layer="1"/>
 </signal>
 </signals>
