File: Hardware/Leiterplatte/Slave/Lixieuhr-Segment.sch (EAGLE design)
At the start: 43 parts, among them U1 APA102C, U10 APA102C, U11 APA102C, U12 APA102C, U13 APA102C, U14 APA102C, U15 APA102C, U16 APA102C, U17 APA102C, U18 APA102C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

Commit message: V06
Parts:
- added C22, C23, C24: 100uF, 0_HTL_MegaCard_V3:CPOL-EUF
- added R1, R2, R3, R4: 0R, 0_HTL_MegaCard_V3:R-R1206
- C21: value 1mF -> 100uF; device rcl:CPOL-USE3.5-8 -> 0_HTL_MegaCard_V3:CPOL-EUF
Connections:
- removed net N$44: JP4.3, U20.DO
- new net N$14: JP1.2, R2.1
- new net N$35: JP1.3, R1.1
- new net N$40: R3.1, U20.CO
- new net N$41: JP4.2, R3.2
- new net N$42: JP4.3, R4.2
- net GND: now also C22.-, C23.-, C24.-
- net N$20: now also R1.2; no longer JP1.3
- net N$43: now also R4.1, U20.DO; no longer JP4.2, U20.CO
- net N$5: now also R2.2; no longer JP1.2
- net V+: now also C22.+, C23.+, C24.+
Other:
- moved on the sheet: JP1, JP4
