File: PCB/Slave/Lixieuhr-Segment.sch (EAGLE design)
At the start: 50 parts, among them U1 APA102C, U10 APA102C, U11 APA102C, U12 APA102C, U13 APA102C, U14 APA102C, U15 APA102C, U16 APA102C, U17 APA102C, U18 APA102C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

Commit message: V05
Parts:
- C21, C22, C23, C24: device 0_HTL_MegaCard_V3:CPOL-EUF -> resistor:CPOL-EU153CLV-0405
Changed lines of the file:
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@@
 <setting verticaltext="up"/>
 </settings>
-<grid distance="0.1" unitdist="inch" unit="inch" style="lines" multiple="1" display="no" altdistance="0.05" altunitdist="inch" altunit="inch"/>
+<grid distance="0.1" unitdist="inch" unit="inch" style="lines" multiple="1" display="no" altdistance="0.01" altunitdist="inch" altunit="inch"/>
 <layers>
 <layer number="1" name="Top" color="4" fill="1" visible="no" active="no"/>
@@
 <part name="P+11" library="0_HTL_analog" deviceset="V+" device=""/>
 <part name="GND43" library="0_HTL_analog" deviceset="GND" device=""/>
-<part name="C21" library="0_HTL_MegaCard_V3" deviceset="CPOL-EU" device="F" value="100uF"/>
-<part name="C22" library="0_HTL_MegaCard_V3" deviceset="CPOL-EU" device="F" value="100uF"/>
-<part name="C23" library="0_HTL_MegaCard_V3" deviceset="CPOL-EU" device="F" value="100uF"/>
-<part name="C24" library="0_HTL_MegaCard_V3" deviceset="CPOL-EU" device="F" value="100uF"/>
+<part name="C21" library="resistor" deviceset="CPOL-EU" device="153CLV-0405" value="100uF"/>
+<part name="C22" library="resistor" deviceset="CPOL-EU" device="153CLV-0405" value="100uF"/>
+<part name="C23" library="resistor" deviceset="CPOL-EU" device="153CLV-0405" value="100uF"/>
+<part name="C24" library="resistor" deviceset="CPOL-EU" device="153CLV-0405" value="100uF"/>
 <part name="R1" library="0_HTL_MegaCard_V3" deviceset="R" device="-R1206" value="0R"/>
 <part name="R2" library="0_HTL_MegaCard_V3" deviceset="R" device="-R1206" value="0R"/>
@@
 <plain>
 <text x="25.4" y="213.36" size="6.4516" layer="105">Lixie-Uhr-Slave</text>
+<wire x1="0" y1="0" x2="279.4" y2="0" width="1.778" layer="100"/>
+<wire x1="279.4" y1="0" x2="279.4" y2="226.06" width="1.778" layer="100"/>
+<wire x1="279.4" y1="226.06" x2="0" y2="226.06" width="1.778" layer="100"/>
+<wire x1="0" y1="226.06" x2="0" y2="0" width="1.778" layer="100"/>
 </plain>
 <instances>
