File: PCB/Slave/Lixieuhr-Segment.brd (EAGLE design)
At the start: 45 x 65 mm, 50 parts, among them U1 APA102C, U10 APA102C, U11 APA102C, U12 APA102C, U13 APA102C, U14 APA102C, U15 APA102C, U16 APA102C, U17 APA102C, U18 APA102C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

Commit message: V05
Parts:
- C21, C22, C23, C24: device 0_HTL_MegaCard_V3:PANASONIC_F -> resistor:153CLV-0405
Routing:
- net GND: track 0.00 -> 174.9 mm, vias 0 -> 15
- net V+: track 304.8 -> 325.6 mm, vias 23 -> 19
- net N$4: track 14.0 -> 11.9 mm

Commit message: V08
Parts:
- moved C11 3.00 mm to (26.0, 30.2), turned to 180 degrees
- moved C1 3.00 mm to (12.5, 47.2)
- moved C10 3.00 mm to (32.8, 31.2)
- moved C12 3.00 mm to (19.2, 30.2)
- moved C13 3.00 mm to (12.5, 23.2)
- moved C14 3.00 mm to (32.8, 23.2)
- moved C15 3.00 mm to (26.0, 22.2), turned to 180 degrees
- moved C16 3.00 mm to (19.2, 22.2)
- moved C17 3.00 mm to (12.5, 15.2)
- moved C18 3.00 mm to (32.8, 15.2)
- moved C19 3.00 mm to (26.0, 14.2), turned to 180 degrees
- moved C2 3.00 mm to (32.8, 47.2)
- moved C20 3.00 mm to (19.2, 14.2)
- moved C3 3.00 mm to (26.0, 46.2), turned to 180 degrees
- moved C4 3.00 mm to (19.2, 46.2)
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Routing:
- net V+: track 325.6 -> 148.1 mm, vias 19 -> 16
- net GND: track 174.9 -> 28.1 mm, vias 15 -> 9
- added copper zone on layer 16, net V+
