File: PCB/Master/Lixie_Master.brd (EAGLE design)
At the start: 52 x 50 mm, 19 parts, among them IC1 FT232RL, J1 65100516121

Commit message: V06
Parts:
- added C4: 0u1, 0_HTL_MegaCard_V3:C0805
- added X1: PIN2", 0_HTL_uC-MEGACARD:PIN2
Connections:
- net GND: now also C4.2, X1.P$2
- net VCC: now also C4.1, X1.P$3
Routing:
- net VCC: track 134.8 -> 141.8 mm
- net N$2: track 14.6 -> 15.7 mm
- net N$14: track 35.0 -> 34.3 mm
- net N$4: track 11.5 -> 10.9 mm

Commit message: V10
Parts:
- added DCF-77: PIN5, 0_HTL_uC-MEGACARD:PIN5
- added R8: (no value), 0_HTL_analog:R0/10
- moved J1 13.0 mm to (34.0, 61.2)
- moved F1 8.90 mm to (43.9, 59.2), turned to 0 degrees
- moved C3 8.14 mm to (49.8, 58.9)
- moved C2 7.38 mm to (55.9, 58.9)
- moved R4 6.68 mm to (32.8, 52.3), turned to 90 degrees
- moved R3 4.58 mm to (35.1, 52.3), turned to 90 degrees
Connections:
- new net N$15: DCF-77.3
- new net N$17: DCF-77.1
- net GND: now also DCF-77.4, R8.1, R8.2
- net PA1: no longer JP1.1
- net PA2: now also DCF-77.2; no longer JP1.3
- net PA3: no longer JP1.5
- net VCC: now also DCF-77.5
Routing:
- net VCC: track 141.8 -> 94.7 mm, vias 3 -> 0
- net PA3: track 25.8 -> 0.00 mm, vias 2 -> 0
- net N$14: track 34.3 -> 10.9 mm, vias 2 -> 0
- net PA1: track 22.6 -> 0.00 mm, vias 2 -> 0
- net PA2: track 22.9 -> 10.7 mm, vias 2 -> 0
- net N$2: track 15.7 -> 6.14 mm, vias 0 -> 2
- net N$4: track 10.9 -> 3.68 mm
- net N$1: track 8.75 -> 4.12 mm
- net N$10: track 10.00 -> 6.80 mm, vias 2 -> 0

Commit message: V10
Parts:
- moved C3 3.05 mm to (52.8, 58.9)
- moved C2 2.29 mm to (58.2, 58.9)
Changed lines of the file:
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@@
 </element>
 <element name="R7" library="0_HTL_analog" package="R0805" value="330" x="70.358" y="48.768" rot="R180"/>
-<element name="C2" library="rcl" package="153CLV-0405" value="4u7" x="55.88" y="58.928" rot="R270"/>
-<element name="C3" library="rcl" package="153CLV-0405" value="4u7" x="49.784" y="58.928" rot="R270"/>
+<element name="C2" library="rcl" package="153CLV-0405" value="4u7" x="58.166" y="58.928" rot="R270"/>
+<element name="C3" library="rcl" package="153CLV-0405" value="4u7" x="52.832" y="58.928" rot="R270"/>
 <element name="F1" library="fuse" package="MF-SMDF050" value="MF-SMDF200" x="43.942" y="59.182"/>
 <element name="X1" library="0_HTL_uC-MEGACARD" package="PIN2" value="PIN2&quot;" x="32.2" y="25.65" rot="R180"/>
@@
 <contactref element="X1" pad="P$3"/>
 <contactref element="C4" pad="1"/>
-<wire x1="55.88" y1="57.128" x2="49.784" y2="57.128" width="0.6096" layer="1"/>
-<wire x1="49.784" y1="57.128" x2="48.446" y2="57.128" width="0.6096" layer="1"/>
 <wire x1="48.446" y1="57.128" x2="46.392" y2="59.182" width="0.6096" layer="1"/>
 <wire x1="30.93" y1="25.65" x2="30.93" y2="27.882" width="0.6096" layer="1"/>
@@
 <wire x1="42.626" y1="29.764" x2="43.688" y2="28.702" width="0.3048" layer="1"/>
 <contactref element="DCF-77" pad="5"/>
-<wire x1="55.88" y1="57.128" x2="59.16" y2="57.128" width="0.6096" layer="1"/>
+<wire x1="64.008" y1="61.976" x2="65.786" y2="61.976" width="0.6096" layer="1"/>
+<wire x1="48.446" y1="57.128" x2="52.832" y2="57.128" width="0.6096" layer="1"/>
+<wire x1="52.832" y1="57.128" x2="58.166" y2="57.128" width="0.6096" layer="1"/>
+<wire x1="58.166" y1="57.128" x2="59.16" y2="57.128" width="0.6096" layer="1"/>
 <wire x1="59.16" y1="57.128" x2="64.008" y2="61.976" width="0.6096" layer="1"/>
-<wire x1="64.008" y1="61.976" x2="65.786" y2="61.976" width="0.6096" layer="1"/>
 </signal>
 <signal name="TXD">

Commit message: V08
Parts:
- renumbered ATTINY-406 to U1
Other:
- board text added: "0.60 mm"
- board text added: "0.80 mm"
- board text added: "0.90 mm"
- board text added: "1.00 mm"
- board text added: "11"
- board text added: "14"
- board text added: "2"
- board text added: "20"
- board text added: "49"
- board text added: "Bohrplan"
- board text added: "CNT"
- board text added: "Material: FR4 1,5mm 35u Cu"
- board text added: "SIZE"
- board text added: "SYM"
- board text added: "TOTAL"
- board text added: "Toleranz: Aussenmass -0,5mm, sonst +/_0,2mm"

Commit message: 080323
Parts:
- added D4: MBRA340T3, diode:SMA
- added R9: 330, 0_HTL_analog:R0805
- R7: value 330 -> 10k
- moved R7 14.1 mm to (57.0, 53.3)
Connections:
- new net N$16: R9.1, S1.3, S1.4
- net N$11: now also D4.C, F1.1; no longer R7.1, S1.3, S1.4
- net N$14: now also D4.A; no longer F1.1
- net RXD: now also U1.8; no longer U1.9
- net TXD: now also U1.9; no longer U1.8
- net UPDI: now also R9.2
- net VCC: now also R7.1
Routing:
- net N$16: track 0.00 -> 13.8 mm
- net PB5: track 47.1 -> 36.2 mm
- net UPDI: track 50.0 -> 58.3 mm
- net N$11: track 13.3 -> 7.12 mm
- net N$14: track 10.9 -> 6.64 mm
- net PA7: track 19.3 -> 23.3 mm
- net GND: track 6.18 -> 9.59 mm, vias 0 -> 2
- net VCC: track 94.7 -> 96.4 mm
- net RXD: track 7.39 -> 7.92 mm, vias 0 -> 2
- net TXD: track 7.08 -> 7.60 mm
