File: PCB/Master/Lixie_Master.sch (EAGLE design)
At the start: 9 parts, among them IC1 FT232RL, J1 65100516121, U1 ATTINY406-MFR

Commit message: V04
Parts:
- removed U1: ATTINY406-MFR, ATTINY406-MFR:ATTINY406-MFR
- added ATTINY-406: (no value), SOIC127P1032X265-20N:ATTINY-406SN
- added JP1: (no value), jumper:JP7Q
- added R3, R4: 27R, 0_HTL_analog:R1206
- added R5, R6: 330R, 0_HTL_analog:R1206
- added S1: TASTER_SMD, 0_HTL_MegaCard_V3:TASTER_SMD
Connections:
- new net N$10: IC1.USBDP, R4.1
- new net N$11: ATTINY-406.PA0/RESET/UPDI, S1.P, S1.P1
- new net N$12: R5.2, U$3.2
- new net N$13: R6.2, U$3.3
- new net N$4: J1.D-, R3.2
- new net PA1: ATTINY-406.PA1, JP1.1
- new net PA2: ATTINY-406.PA2, JP1.3
- new net PA3: ATTINY-406.EXTCLK/PA3, JP1.5
- new net PA4: JP1.7
- new net PA5: JP1.9
- new net PA6: ATTINY-406.PA6, JP1.11
- new net PA7: ATTINY-406.PA7, JP1.13
- new net PB0: ATTINY-406.PB0, JP1.2
- new net PB1: ATTINY-406.PB1, JP1.4
- new net PB4: ATTINY-406.PA4, ATTINY-406.PB4, JP1.6
- new net PB5: ATTINY-406.PA5, ATTINY-406.PB5, JP1.8
- new net PC1: ATTINY-406.PC1, JP1.10
- new net PC3: ATTINY-406.PC3, JP1.12
- net GND: now also ATTINY-406.GND, JP1.14; no longer U1.GND
- net N$1: now also R4.2; no longer IC1.USBDP
- net N$2: now also R3.1; no longer J1.D-
- net N$8: now also ATTINY-406.PC0, R5.1; no longer U$3.2, U1.PC0
- net N$9: now also ATTINY-406.PC2, R6.1; no longer U$3.3, U1.PC2
- net RXD: now also ATTINY-406.PB2, IC1.TXD; no longer IC1.RXD, U1.PB3
- net TXD: now also ATTINY-406.PB3, IC1.RXD; no longer IC1.TXD, U1.PB2
- net VCC: now also ATTINY-406.VDD, S1.S, S1.S1; no longer U1.VDD
Other:
- moved on the sheet: C1, D1, D2, IC1, J1, R1, R2, U$3

Commit message: Master
Parts:
- added C2, C3: 4u7, rcl:CPOL-EU153CLV-0405
- added F1: MF-SMDF200, fuse:MF-SMDF200
- added R7: 330, 0_HTL_analog:R0805
Connections:
- new net N$14: F1.1, J1.VBUS
- new net UPDI: ATTINY-406.PA0/RESET/UPDI, JP1.14, R7.2
- net GND: now also C2.-, C3.-, S1.S, S1.S1; no longer JP1.14
- net N$11: now also R7.1; no longer ATTINY-406.PA0/RESET/UPDI
- net VCC: now also C2.+, C3.+, F1.2; no longer J1.VBUS, S1.S, S1.S1

Commit message: V06
Parts:
- added C4: 0u1, 0_HTL_MegaCard_V3:C-EUC0805
- added X1: PIN2", 0_HTL_uC-MEGACARD:PIN2"
Connections:
- net GND: now also C4.2, X1.KL1
- net VCC: now also C4.1, X1.KL2
Changed lines of the file:
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@@
 <part name="C3" library="rcl" deviceset="CPOL-EU" device="153CLV-0405" value="4u7"/>
 <part name="F1" library="fuse" deviceset="MF-SMDF" device="" technology="200"/>
+<part name="X1" library="0_HTL_uC-MEGACARD" deviceset="PIN2" device="&quot;"/>
+<part name="U$5" library="0_HTL_analog_neu" deviceset="VCC" device=""/>
+<part name="GND8" library="0_HTL_analog_neu" deviceset="GND" device=""/>
+<part name="C4" library="0_HTL_MegaCard_V3" deviceset="C-EU" device="C0805" value="0u1"/>
 </parts>
 <sheets>
@@
 <instance part="C3" gate="G$1" x="233.68" y="78.74"/>
 <instance part="F1" gate="A" x="27.94" y="66.04" rot="R90"/>
+<instance part="X1" gate="G$2" x="5.08" y="76.2" rot="R90"/>
+<instance part="U$5" gate="G$1" x="10.16" y="86.36"/>
+<instance part="GND8" gate="1" x="10.16" y="71.12"/>
+<instance part="C4" gate="G$1" x="175.26" y="81.28" rot="R270"/>
 </instances>
 <busses>
@@
 <pinref part="S1" gate="G$1" pin="S1"/>
 <wire x1="142.24" y1="81.28" x2="144.78" y2="81.28" width="0.1524" layer="91"/>
+<pinref part="C4" gate="G$1" pin="2"/>
+<wire x1="170.18" y1="81.28" x2="167.64" y2="81.28" width="0.1524" layer="91"/>
+<junction x="167.64" y="81.28"/>
 </segment>
 <segment>
@@
 <wire x1="233.68" y1="71.12" x2="233.68" y2="73.66" width="0.1524" layer="91"/>
 <junction x="226.06" y="71.12"/>
+</segment>
+<segment>
+<pinref part="X1" gate="G$2" pin="KL1"/>
+<pinref part="GND8" gate="1" pin="GND"/>
+<wire x1="5.08" y1="76.2" x2="10.16" y2="76.2" width="0.1524" layer="91"/>
+<wire x1="10.16" y1="76.2" x2="10.16" y2="73.66" width="0.1524" layer="91"/>
 </segment>
 </net>
@@
 <wire x1="203.2" y1="71.12" x2="203.2" y2="81.28" width="0.1524" layer="91"/>
 <pinref part="ATTINY-406" gate="G$1" pin="VDD"/>
+<pinref part="C4" gate="G$1" pin="1"/>
+<wire x1="177.8" y1="81.28" x2="180.34" y2="81.28" width="0.1524" layer="91"/>
+<junction x="180.34" y="81.28"/>
 </segment>
 <segment>
@@
 <junction x="226.06" y="83.82"/>
 </segment>
-</net>
+<segment>
+<pinref part="X1" gate="G$2" pin="KL2"/>
+<pinref part="U$5" gate="G$1" pin="VCC"/>
+<wire x1="5.08" y1="78.74" x2="10.16" y2="78.74" width="0.1524" layer="91"/>
+<wire x1="10.16" y1="78.74" x2="10.16" y2="81.28" width="0.1524" layer="91"/>
+</segment>
+</net>

Commit message: V10
Parts:
- added DCF-77: PIN5, 0_HTL_uC-MEGACARD:PIN5
- added R8: (no value), 0_HTL_analog:R0/10
Connections:
- new net N$15: DCF-77.3
- new net N$17: DCF-77.1
- net GND: now also DCF-77.4, R8.1, R8.2
- net PA1: no longer JP1.1
- net PA2: now also DCF-77.2; no longer JP1.3
- net PA3: no longer JP1.5
- net VCC: now also DCF-77.5
Other:
- moved on the sheet: JP1
Changed lines of the file:
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@@
 <part name="GND8" library="0_HTL_analog_neu" deviceset="GND" device=""/>
 <part name="C4" library="0_HTL_MegaCard_V3" deviceset="C-EU" device="C0805" value="0u1"/>
+<part name="DCF-77" library="0_HTL_uC-MEGACARD" deviceset="PIN5" device=""/>
+<part name="U$7" library="0_HTL_analog_neu" deviceset="VCC" device=""/>
+<part name="GND9" library="0_HTL_analog_neu" deviceset="GND" device=""/>
+<part name="R8" library="0_HTL_analog" deviceset="R0" device="/10"/>
+<part name="GND10" library="0_HTL_analog_neu" deviceset="GND" device=""/>
+<part name="GND11" library="0_HTL_analog_neu" deviceset="GND" device=""/>
 </parts>
 <sheets>
@@
 <attribute name="VALUE" x="209.55" y="61.468" size="1.778" layer="96"/>
 </instance>
-<instance part="JP1" gate="B" x="259.08" y="50.8" rot="R90"/>
+<instance part="JP1" gate="B" x="114.3" y="2.54" rot="R90"/>
 <instance part="ATTINY-406" gate="G$1" x="154.94" y="48.26"/>
 <instance part="R7" gate="G$1" x="129.54" y="73.66" rot="R180"/>
@@
 <instance part="GND8" gate="1" x="10.16" y="71.12"/>
 <instance part="C4" gate="G$1" x="175.26" y="81.28" rot="R270"/>
+<instance part="DCF-77" gate="G$1" x="2.54" y="25.4" rot="R90"/>
+<instance part="U$7" gate="G$1" x="17.78" y="43.18"/>
+<instance part="GND9" gate="1" x="17.78" y="27.94"/>
+<instance part="R8" gate="G$1" x="106.68" y="30.48"/>
+<instance part="GND10" gate="1" x="101.6" y="25.4"/>
+<instance part="GND11" gate="1" x="111.76" y="25.4"/>
 </instances>
 <busses>
@@
 <wire x1="5.08" y1="76.2" x2="10.16" y2="76.2" width="0.1524" layer="91"/>
 <wire x1="10.16" y1="76.2" x2="10.16" y2="73.66" width="0.1524" layer="91"/>
+</segment>
+<segment>
+<pinref part="GND9" gate="1" pin="GND"/>
+<pinref part="DCF-77" gate="G$1" pin="4"/>
+<wire x1="2.54" y1="33.02" x2="17.78" y2="33.02" width="0.1524" layer="91"/>
+<wire x1="17.78" y1="33.02" x2="17.78" y2="30.48" width="0.1524" layer="91"/>
+</segment>
+<segment>
+<pinref part="GND10" gate="1" pin="GND"/>
+<wire x1="101.6" y1="27.94" x2="101.6" y2="30.48" width="0.1524" layer="91"/>
+<pinref part="R8" gate="G$1" pin="1"/>
+<wire x1="101.6" y1="30.48" x2="104.14" y2="30.48" width="0.1524" layer="91"/>
+</segment>
+<segment>
+<pinref part="R8" gate="G$1" pin="2"/>
+<pinref part="GND11" gate="1" pin="GND"/>
+<wire x1="109.22" y1="30.48" x2="111.76" y2="30.48" width="0.1524" layer="91"/>
+<wire x1="111.76" y1="30.48" x2="111.76" y2="27.94" width="0.1524" layer="91"/>
 </segment>
 </net>
@@
 <wire x1="10.16" y1="78.74" x2="10.16" y2="81.28" width="0.1524" layer="91"/>
 </segment>
+<segment>
+<pinref part="U$7" gate="G$1" pin="VCC"/>
+<wire x1="17.78" y1="35.56" x2="17.78" y2="38.1" width="0.1524" layer="91"/>
+<pinref part="DCF-77" gate="G$1" pin="5"/>
+<wire x1="2.54" y1="35.56" x2="17.78" y2="35.56" width="0.1524" layer="91"/>
+</segment>
 </net>
 <net name="TXD" class="0">
@@
 <segment>
 <pinref part="JP1" gate="B" pin="14"/>
-<wire x1="251.46" y1="58.42" x2="226.06" y2="58.42" width="0.1524" layer="91"/>
-<label x="226.06" y="58.42" size="1.778" layer="95" rot="R270" xref="yes"/>
+<wire x1="106.68" y1="10.16" x2="81.28" y2="10.16" width="0.1524" layer="91"/>
+<label x="81.28" y="10.16" size="1.778" layer="95" rot="R270" xref="yes"/>
 </segment>
 </net>
@@
 <segment>
 <pinref part="JP1" gate="B" pin="11"/>
-<wire x1="266.7" y1="55.88" x2="288.29" y2="55.88" width="0.1524" layer="91"/>
-<label x="288.29" y="55.88" size="1.778" layer="95" rot="R270" xref="yes"/>
+<wire x1="121.92" y1="7.62" x2="143.51" y2="7.62" width="0.1524" layer="91"/>
+<label x="143.51" y="7.62" size="1.778" layer="95" rot="R270" xref="yes"/>
 </segment>
 </net>
@@
 <segment>
 <pinref part="JP1" gate="B" pin="13"/>
-<wire x1="266.7" y1="58.42" x2="292.1" y2="58.42" width="0.1524" layer="91"/>
-<label x="292.1" y="58.42" size="1.778" layer="95" rot="R270" xref="yes"/>
+<wire x1="121.92" y1="10.16" x2="147.32" y2="10.16" width="0.1524" layer="91"/>
+<label x="147.32" y="10.16" size="1.778" layer="95" rot="R270" xref="yes"/>
 </segment>
 </net>
@@
 <segment>
 <pinref part="JP1" gate="B" pin="6"/>
-<wire x1="251.46" y1="48.26" x2="241.3" y2="48.26" width="0.1524" layer="91"/>
-<label x="241.3" y="48.26" size="1.778" layer="95" rot="R270" xref="yes"/>
+<wire x1="106.68" y1="0" x2="96.52" y2="0" width="0.1524" layer="91"/>
+<label x="96.52" y="0" size="1.778" layer="95" rot="R270" xref="yes"/>
 </segment>
 </net>
@@
 <segment>
 <pinref part="JP1" gate="B" pin="8"/>
-<wire x1="251.46" y1="50.8" x2="237.49" y2="50.8" width="0.1524" layer="91"/>
-<label x="237.49" y="50.8" size="1.778" layer="95" rot="R270" xref="yes"/>
+<wire x1="106.68" y1="2.54" x2="92.71" y2="2.54" width="0.1524" layer="91"/>
+<label x="92.71" y="2.54" size="1.778" layer="95" rot="R270" xref="yes"/>
 </segment>
 </net>
@@
 <segment>
 <pinref part="JP1" gate="B" pin="12"/>
-<wire x1="251.46" y1="55.88" x2="229.87" y2="55.88" width="0.1524" layer="91"/>
-<label x="229.87" y="55.88" size="1.778" layer="95" rot="R270" xref="yes"/>
+<wire x1="106.68" y1="7.62" x2="85.09" y2="7.62" width="0.1524" layer="91"/>
+<label x="85.09" y="7.62" size="1.778" layer="95" rot="R270" xref="yes"/>
 </segment>
 </net>
@@
 <pinref part="ATTINY-406" gate="G$1" pin="PA1"/>
 </segment>
-<segment>
-<pinref part="JP1" gate="B" pin="1"/>
-<wire x1="266.7" y1="43.18" x2="269.24" y2="43.18" width="0.1524" layer="91"/>
-<label x="269.24" y="43.18" size="1.778" layer="95" rot="R270" xref="yes"/>
-</segment>
 </net>
 <net name="PA2" class="0">
@@
 </segment>
 <segment>
-<pinref part="JP1" gate="B" pin="3"/>
-<wire x1="266.7" y1="45.72" x2="273.05" y2="45.72" width="0.1524" layer="91"/>
-<label x="273.05" y="45.72" size="1.778" layer="95" rot="R270" xref="yes"/>
+<pinref part="DCF-77" gate="G$1" pin="2"/>
+<wire x1="2.54" y1="27.94" x2="7.62" y2="27.94" width="0.1524" layer="91"/>
+<label x="7.62" y="27.94" size="1.778" layer="95" xref="yes"/>
 </segment>
 </net>
@@
 <pinref part="ATTINY-406" gate="G$1" pin="EXTCLK/PA3"/>
 </segment>
-<segment>
-<pinref part="JP1" gate="B" pin="5"/>
-<wire x1="266.7" y1="48.26" x2="276.86" y2="48.26" width="0.1524" layer="91"/>
-<label x="276.86" y="48.26" size="1.778" layer="95" rot="R270" xref="yes"/>
-</segment>
 </net>
 <net name="PB0" class="0">
@@
 <segment>
 <pinref part="JP1" gate="B" pin="2"/>
-<wire x1="251.46" y1="43.18" x2="248.92" y2="43.18" width="0.1524" layer="91"/>
-<label x="248.92" y="43.18" size="1.778" layer="95" rot="R270" xref="yes"/>
+<wire x1="106.68" y1="-5.08" x2="104.14" y2="-5.08" width="0.1524" layer="91"/>
+<label x="104.14" y="-5.08" size="1.778" layer="95" rot="R270" xref="yes"/>
 </segment>
 </net>
@@
 <segment>
 <pinref part="JP1" gate="B" pin="4"/>
-<wire x1="251.46" y1="45.72" x2="245.11" y2="45.72" width="0.1524" layer="91"/>
-<label x="245.11" y="45.72" size="1.778" layer="95" rot="R270" xref="yes"/>
+<wire x1="106.68" y1="-2.54" x2="100.33" y2="-2.54" width="0.1524" layer="91"/>
+<label x="100.33" y="-2.54" size="1.778" layer="95" rot="R270" xref="yes"/>
 </segment>
 </net>
@@
 <segment>
 <pinref part="JP1" gate="B" pin="10"/>
-<wire x1="251.46" y1="53.34" x2="233.68" y2="53.34" width="0.1524" layer="91"/>
-<label x="233.68" y="53.34" size="1.778" layer="95" rot="R270" xref="yes"/>
+<wire x1="106.68" y1="5.08" x2="88.9" y2="5.08" width="0.1524" layer="91"/>
+<label x="88.9" y="5.08" size="1.778" layer="95" rot="R270" xref="yes"/>
 </segment>
 </net>
@@
 <segment>
 <pinref part="JP1" gate="B" pin="7"/>
-<wire x1="266.7" y1="50.8" x2="280.67" y2="50.8" width="0.1524" layer="91"/>
-<label x="280.67" y="50.8" size="1.778" layer="95" rot="R270" xref="yes"/>
+<wire x1="121.92" y1="2.54" x2="135.89" y2="2.54" width="0.1524" layer="91"/>
+<label x="135.89" y="2.54" size="1.778" layer="95" rot="R270" xref="yes"/>
 </segment>
 </net>
@@
 <segment>
 <pinref part="JP1" gate="B" pin="9"/>
-<wire x1="266.7" y1="53.34" x2="284.48" y2="53.34" width="0.1524" layer="91"/>
-<label x="284.48" y="53.34" size="1.778" layer="95" rot="R270" xref="yes"/>
+<wire x1="121.92" y1="5.08" x2="139.7" y2="5.08" width="0.1524" layer="91"/>
+<label x="139.7" y="5.08" size="1.778" layer="95" rot="R270" xref="yes"/>
 </segment>
 </net>
@@
 </segment>
 </net>
+<net name="N$15" class="0">
+<segment>
+<pinref part="DCF-77" gate="G$1" pin="3"/>
+<wire x1="2.54" y1="30.48" x2="7.62" y2="30.48" width="0.1524" layer="91"/>
+</segment>
+</net>
+<net name="N$17" class="0">
+<segment>
+<pinref part="DCF-77" gate="G$1" pin="1"/>
+<wire x1="2.54" y1="25.4" x2="7.62" y2="25.4" width="0.1524" layer="91"/>
+</segment>
+</net>
 </nets>
 </sheet>
 </sheets>
+<errors>
+</errors>
 </schematic>
 </drawing>

Commit message: V08
Parts:
- renumbered ATTINY-406 to U1
Changed lines of the file:
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@@
 <part name="R6" library="0_HTL_analog" deviceset="R" device="1206" value="330R"/>
 <part name="JP1" library="jumper" deviceset="JP7Q" device=""/>
-<part name="ATTINY-406" library="SOIC127P1032X265-20N" deviceset="ATTINY-406SN" device=""/>
+<part name="U1" library="SOIC127P1032X265-20N" deviceset="ATTINY-406SN" device=""/>
 <part name="R7" library="0_HTL_analog" deviceset="R" device="0805" value="330"/>
 <part name="GND6" library="0_HTL_analog_neu" deviceset="GND" device=""/>
@@
 </instance>
 <instance part="JP1" gate="B" x="114.3" y="2.54" rot="R90"/>
-<instance part="ATTINY-406" gate="G$1" x="154.94" y="48.26"/>
+<instance part="U1" gate="G$1" x="154.94" y="48.26"/>
 <instance part="R7" gate="G$1" x="129.54" y="73.66" rot="R180"/>
 <instance part="GND6" gate="1" x="167.64" y="76.2"/>
@@
 <pinref part="U$3" gate="G$1" pin="4"/>
 <wire x1="210.82" y1="33.02" x2="210.82" y2="81.28" width="0.1524" layer="91"/>
-<pinref part="ATTINY-406" gate="G$1" pin="GND"/>
+<pinref part="U1" gate="G$1" pin="GND"/>
 <wire x1="175.26" y1="33.02" x2="180.34" y2="33.02" width="0.1524" layer="91"/>
 <pinref part="GND5" gate="1" pin="GND"/>
@@
 <wire x1="180.34" y1="71.12" x2="203.2" y2="71.12" width="0.1524" layer="91"/>
 <wire x1="203.2" y1="71.12" x2="203.2" y2="81.28" width="0.1524" layer="91"/>
-<pinref part="ATTINY-406" gate="G$1" pin="VDD"/>
+<pinref part="U1" gate="G$1" pin="VDD"/>
 <pinref part="C4" gate="G$1" pin="1"/>
 <wire x1="177.8" y1="81.28" x2="180.34" y2="81.28" width="0.1524" layer="91"/>
@@
 <wire x1="175.26" y1="53.34" x2="180.34" y2="53.34" width="0.1524" layer="91"/>
 <label x="180.34" y="53.34" size="1.778" layer="95" xref="yes"/>
-<pinref part="ATTINY-406" gate="G$1" pin="PB3"/>
+<pinref part="U1" gate="G$1" pin="PB3"/>
 </segment>
 </net>
@@
 <wire x1="134.62" y1="48.26" x2="121.92" y2="48.26" width="0.1524" layer="91"/>
 <label x="121.92" y="48.26" size="1.778" layer="95" rot="R180" xref="yes"/>
-<pinref part="ATTINY-406" gate="G$1" pin="PB2"/>
+<pinref part="U1" gate="G$1" pin="PB2"/>
 </segment>
 </net>
@@
 <wire x1="205.74" y1="20.32" x2="205.74" y2="58.42" width="0.1524" layer="91"/>
 <pinref part="R5" gate="G$1" pin="1"/>
-<pinref part="ATTINY-406" gate="G$1" pin="PC0"/>
+<pinref part="U1" gate="G$1" pin="PC0"/>
 </segment>
 </net>
@@
 <wire x1="208.28" y1="43.18" x2="208.28" y2="58.42" width="0.1524" layer="91"/>
 <pinref part="R6" gate="G$1" pin="1"/>
-<pinref part="ATTINY-406" gate="G$1" pin="PC2"/>
+<pinref part="U1" gate="G$1" pin="PC2"/>
 </segment>
 </net>
@@
 <net name="UPDI" class="0">
 <segment>
-<pinref part="ATTINY-406" gate="G$1" pin="PA0/RESET/UPDI"/>
+<pinref part="U1" gate="G$1" pin="PA0/RESET/UPDI"/>
 <wire x1="134.62" y1="66.04" x2="129.54" y2="66.04" width="0.1524" layer="91"/>
 <label x="121.92" y="66.04" size="1.778" layer="95" rot="R180" xref="yes"/>
@@
 <wire x1="175.26" y1="60.96" x2="180.34" y2="60.96" width="0.1524" layer="91"/>
 <label x="180.34" y="60.96" size="1.778" layer="95" xref="yes"/>
-<pinref part="ATTINY-406" gate="G$1" pin="PA6"/>
+<pinref part="U1" gate="G$1" pin="PA6"/>
 </segment>
 <segment>
@@
 <label x="187.96" y="58.42" size="1.778" layer="95" xref="yes"/>
 <wire x1="187.96" y1="58.42" x2="175.26" y2="58.42" width="0.1524" layer="91"/>
-<pinref part="ATTINY-406" gate="G$1" pin="PA7"/>
+<pinref part="U1" gate="G$1" pin="PA7"/>
 </segment>
 <segment>
@@
 <label x="187.96" y="50.8" size="1.778" layer="95" xref="yes"/>
 <wire x1="175.26" y1="50.8" x2="187.96" y2="50.8" width="0.1524" layer="91"/>
-<pinref part="ATTINY-406" gate="G$1" pin="PB4"/>
+<pinref part="U1" gate="G$1" pin="PB4"/>
 </segment>
 <segment>
 <wire x1="175.26" y1="66.04" x2="180.34" y2="66.04" width="0.1524" layer="91"/>
 <label x="180.34" y="66.04" size="1.778" layer="95" xref="yes"/>
-<pinref part="ATTINY-406" gate="G$1" pin="PA4"/>
+<pinref part="U1" gate="G$1" pin="PA4"/>
 </segment>
 <segment>
@@
 <wire x1="175.26" y1="48.26" x2="180.34" y2="48.26" width="0.1524" layer="91"/>
 <label x="180.34" y="48.26" size="1.778" layer="95" xref="yes"/>
-<pinref part="ATTINY-406" gate="G$1" pin="PB5"/>
+<pinref part="U1" gate="G$1" pin="PB5"/>
 </segment>
 <segment>
 <label x="187.96" y="63.5" size="1.778" layer="95" xref="yes"/>
 <wire x1="175.26" y1="63.5" x2="187.96" y2="63.5" width="0.1524" layer="91"/>
-<pinref part="ATTINY-406" gate="G$1" pin="PA5"/>
+<pinref part="U1" gate="G$1" pin="PA5"/>
 </segment>
 <segment>
@@
 <wire x1="175.26" y1="40.64" x2="180.34" y2="40.64" width="0.1524" layer="91"/>
 <label x="180.34" y="40.64" size="1.778" layer="95" xref="yes"/>
-<pinref part="ATTINY-406" gate="G$1" pin="PC3"/>
+<pinref part="U1" gate="G$1" pin="PC3"/>
 </segment>
 <segment>
@@
 <wire x1="134.62" y1="63.5" x2="129.54" y2="63.5" width="0.1524" layer="91"/>
 <label x="129.54" y="63.5" size="1.778" layer="95" rot="R180" xref="yes"/>
-<pinref part="ATTINY-406" gate="G$1" pin="PA1"/>
+<pinref part="U1" gate="G$1" pin="PA1"/>
 </segment>
 </net>
@@
 <wire x1="134.62" y1="60.96" x2="121.92" y2="60.96" width="0.1524" layer="91"/>
 <label x="121.92" y="60.96" size="1.778" layer="95" rot="R180" xref="yes"/>
-<pinref part="ATTINY-406" gate="G$1" pin="PA2"/>
+<pinref part="U1" gate="G$1" pin="PA2"/>
 </segment>
 <segment>
@@
 <wire x1="134.62" y1="58.42" x2="129.54" y2="58.42" width="0.1524" layer="91"/>
 <label x="129.54" y="58.42" size="1.778" layer="95" rot="R180" xref="yes"/>
-<pinref part="ATTINY-406" gate="G$1" pin="EXTCLK/PA3"/>
+<pinref part="U1" gate="G$1" pin="EXTCLK/PA3"/>
 </segment>
 </net>
@@
 <wire x1="134.62" y1="53.34" x2="121.92" y2="53.34" width="0.1524" layer="91"/>
 <label x="121.92" y="53.34" size="1.778" layer="95" rot="R180" xref="yes"/>
-<pinref part="ATTINY-406" gate="G$1" pin="PB0"/>
+<pinref part="U1" gate="G$1" pin="PB0"/>
 </segment>
 <segment>
@@
 <wire x1="134.62" y1="50.8" x2="129.54" y2="50.8" width="0.1524" layer="91"/>
 <label x="129.54" y="50.8" size="1.778" layer="95" rot="R180" xref="yes"/>
-<pinref part="ATTINY-406" gate="G$1" pin="PB1"/>
+<pinref part="U1" gate="G$1" pin="PB1"/>
 </segment>
 <segment>
@@
 <wire x1="134.62" y1="40.64" x2="129.54" y2="40.64" width="0.1524" layer="91"/>
 <label x="129.54" y="40.64" size="1.778" layer="95" rot="R180" xref="yes"/>
-<pinref part="ATTINY-406" gate="G$1" pin="PC1"/>
-</segment>
-<segment>
+<pinref part="U1" gate="G$1" pin="PC1"/>
+</segment>
+<segment>
