File: PCB/Master/Lixie_Master.sch (EAGLE design)
At the start: 23 parts, among them IC1 FT232RL, J1 65100516121, X1 PIN2"

Commit message: 080323
Parts:
- added D4: MBRA340T3, diode:MBRA340T3
- added R9: 330, 0_HTL_analog:R0805
- R7: value 330 -> 10k
Connections:
- new net N$16: R9.1, S1.P, S1.P1
- net N$11: now also D4.C, F1.1; no longer R7.1, S1.P, S1.P1
- net N$14: now also D4.A; no longer F1.1
- net RXD: now also U1.PB3; no longer U1.PB2
- net TXD: now also U1.PB2; no longer U1.PB3
- net UPDI: now also R9.2
- net VCC: now also R7.1
Other:
- moved on the sheet: R7, S1
Changed lines of the file:
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@@
 <part name="JP1" library="jumper" deviceset="JP7Q" device=""/>
 <part name="U1" library="SOIC127P1032X265-20N" deviceset="ATTINY-406SN" device=""/>
-<part name="R7" library="0_HTL_analog" deviceset="R" device="0805" value="330"/>
+<part name="R7" library="0_HTL_analog" deviceset="R" device="0805" value="10k"/>
 <part name="GND6" library="0_HTL_analog_neu" deviceset="GND" device=""/>
 <part name="U$4" library="0_HTL_analog_neu" deviceset="VCC" device=""/>
@@
 <part name="GND10" library="0_HTL_analog_neu" deviceset="GND" device=""/>
 <part name="GND11" library="0_HTL_analog_neu" deviceset="GND" device=""/>
+<part name="U$6" library="0_HTL_analog_neu" deviceset="VCC" device=""/>
+<part name="R9" library="0_HTL_analog" deviceset="R" device="0805" value="330"/>
+<part name="GND12" library="0_HTL_analog_neu" deviceset="GND" device=""/>
+<part name="D4" library="diode" deviceset="MBRA340T3" device=""/>
 </parts>
 <sheets>
@@
 <attribute name="VALUE" x="36.83" y="43.688" size="1.778" layer="96"/>
 </instance>
-<instance part="S1" gate="G$1" x="137.16" y="83.82" rot="R270"/>
+<instance part="S1" gate="G$1" x="121.92" y="88.9"/>
 <instance part="R5" gate="G$1" x="205.74" y="63.5" smashed="yes">
 <attribute name="NAME" x="204.47" y="65.8114" size="1.778" layer="95" rot="R180"/>
@@
 <instance part="JP1" gate="B" x="114.3" y="2.54" rot="R90"/>
 <instance part="U1" gate="G$1" x="154.94" y="48.26"/>
-<instance part="R7" gate="G$1" x="129.54" y="73.66" rot="R180"/>
+<instance part="R7" gate="G$1" x="129.54" y="81.28" rot="R180"/>
 <instance part="GND6" gate="1" x="167.64" y="76.2"/>
 <instance part="U$4" gate="G$1" x="226.06" y="88.9"/>
@@
 <instance part="GND10" gate="1" x="101.6" y="25.4"/>
 <instance part="GND11" gate="1" x="111.76" y="25.4"/>
+<instance part="U$6" gate="G$1" x="129.54" y="93.98"/>
+<instance part="R9" gate="G$1" x="124.46" y="73.66" rot="R180"/>
+<instance part="GND12" gate="1" x="121.92" y="101.6" rot="R180"/>
+<instance part="D4" gate="G$1" x="33.02" y="60.96" rot="R90"/>
 </instances>
 <busses>
@@
 </segment>
 <segment>
+<pinref part="C4" gate="G$1" pin="2"/>
+<wire x1="170.18" y1="81.28" x2="167.64" y2="81.28" width="0.1524" layer="91"/>
 <pinref part="GND6" gate="1" pin="GND"/>
 <wire x1="167.64" y1="78.74" x2="167.64" y2="81.28" width="0.1524" layer="91"/>
-<pinref part="S1" gate="G$1" pin="S"/>
-<wire x1="144.78" y1="83.82" x2="142.24" y2="83.82" width="0.1524" layer="91"/>
-<wire x1="144.78" y1="81.28" x2="144.78" y2="83.82" width="0.1524" layer="91"/>
-<wire x1="144.78" y1="81.28" x2="167.64" y2="81.28" width="0.1524" layer="91"/>
-<junction x="144.78" y="81.28"/>
-<pinref part="S1" gate="G$1" pin="S1"/>
-<wire x1="142.24" y1="81.28" x2="144.78" y2="81.28" width="0.1524" layer="91"/>
-<pinref part="C4" gate="G$1" pin="2"/>
-<wire x1="170.18" y1="81.28" x2="167.64" y2="81.28" width="0.1524" layer="91"/>
-<junction x="167.64" y="81.28"/>
 </segment>
 <segment>
@@
 <wire x1="109.22" y1="30.48" x2="111.76" y2="30.48" width="0.1524" layer="91"/>
 <wire x1="111.76" y1="30.48" x2="111.76" y2="27.94" width="0.1524" layer="91"/>
+</segment>
+<segment>
+<pinref part="S1" gate="G$1" pin="S1"/>
+<wire x1="124.46" y1="93.98" x2="124.46" y2="96.52" width="0.1524" layer="91"/>
+<wire x1="124.46" y1="96.52" x2="121.92" y2="96.52" width="0.1524" layer="91"/>
+<pinref part="S1" gate="G$1" pin="S"/>
+<wire x1="121.92" y1="96.52" x2="121.92" y2="93.98" width="0.1524" layer="91"/>
+<pinref part="GND12" gate="1" pin="GND"/>
+<wire x1="121.92" y1="96.52" x2="121.92" y2="99.06" width="0.1524" layer="91"/>
+<junction x="121.92" y="96.52"/>
 </segment>
 </net>
@@
 </segment>
 <segment>
-<pinref part="X1" gate="G$2" pin="KL2"/>
-<pinref part="U$5" gate="G$1" pin="VCC"/>
-<wire x1="5.08" y1="78.74" x2="10.16" y2="78.74" width="0.1524" layer="91"/>
-<wire x1="10.16" y1="78.74" x2="10.16" y2="81.28" width="0.1524" layer="91"/>
-</segment>
-<segment>
 <pinref part="U$7" gate="G$1" pin="VCC"/>
 <wire x1="17.78" y1="35.56" x2="17.78" y2="38.1" width="0.1524" layer="91"/>
@@
 <wire x1="2.54" y1="35.56" x2="17.78" y2="35.56" width="0.1524" layer="91"/>
 </segment>
+<segment>
+<pinref part="R7" gate="G$1" pin="1"/>
+<wire x1="129.54" y1="86.36" x2="129.54" y2="88.9" width="0.1524" layer="91"/>
+<pinref part="U$6" gate="G$1" pin="VCC"/>
+</segment>
+<segment>
+<pinref part="X1" gate="G$2" pin="KL2"/>
+<wire x1="5.08" y1="78.74" x2="10.16" y2="78.74" width="0.1524" layer="91"/>
+<pinref part="U$5" gate="G$1" pin="VCC"/>
+<wire x1="10.16" y1="78.74" x2="10.16" y2="81.28" width="0.1524" layer="91"/>
+</segment>
 </net>
 <net name="TXD" class="0">
@@
 </segment>
 <segment>
-<wire x1="175.26" y1="53.34" x2="180.34" y2="53.34" width="0.1524" layer="91"/>
-<label x="180.34" y="53.34" size="1.778" layer="95" xref="yes"/>
-<pinref part="U1" gate="G$1" pin="PB3"/>
+<wire x1="134.62" y1="48.26" x2="121.92" y2="48.26" width="0.1524" layer="91"/>
+<label x="121.92" y="48.26" size="1.778" layer="95" rot="R180" xref="yes"/>
+<pinref part="U1" gate="G$1" pin="PB2"/>
 </segment>
 </net>
@@
 </segment>
 <segment>
-<wire x1="134.62" y1="48.26" x2="121.92" y2="48.26" width="0.1524" layer="91"/>
-<label x="121.92" y="48.26" size="1.778" layer="95" rot="R180" xref="yes"/>
-<pinref part="U1" gate="G$1" pin="PB2"/>
+<wire x1="175.26" y1="53.34" x2="180.34" y2="53.34" width="0.1524" layer="91"/>
+<label x="180.34" y="53.34" size="1.778" layer="95" xref="yes"/>
+<pinref part="U1" gate="G$1" pin="PB3"/>
 </segment>
 </net>
@@
 <label x="121.92" y="66.04" size="1.778" layer="95" rot="R180" xref="yes"/>
 <pinref part="R7" gate="G$1" pin="2"/>
-<wire x1="129.54" y1="66.04" x2="121.92" y2="66.04" width="0.1524" layer="91"/>
-<wire x1="129.54" y1="68.58" x2="129.54" y2="66.04" width="0.1524" layer="91"/>
+<wire x1="129.54" y1="66.04" x2="124.46" y2="66.04" width="0.1524" layer="91"/>
+<wire x1="124.46" y1="66.04" x2="121.92" y2="66.04" width="0.1524" layer="91"/>
+<wire x1="129.54" y1="76.2" x2="129.54" y2="66.04" width="0.1524" layer="91"/>
 <junction x="129.54" y="66.04"/>
+<pinref part="R9" gate="G$1" pin="2"/>
+<wire x1="124.46" y1="68.58" x2="124.46" y2="66.04" width="0.1524" layer="91"/>
+<junction x="124.46" y="66.04"/>
 </segment>
 <segment>
@@
 </segment>
 </net>
-<net name="N$11" class="0">
-<segment>
-<pinref part="S1" gate="G$1" pin="P1"/>
-<wire x1="129.54" y1="81.28" x2="132.08" y2="81.28" width="0.1524" layer="91"/>
-<pinref part="S1" gate="G$1" pin="P"/>
-<wire x1="132.08" y1="83.82" x2="129.54" y2="83.82" width="0.1524" layer="91"/>
-<wire x1="129.54" y1="83.82" x2="129.54" y2="81.28" width="0.1524" layer="91"/>
-<pinref part="R7" gate="G$1" pin="1"/>
-<wire x1="129.54" y1="81.28" x2="129.54" y2="78.74" width="0.1524" layer="91"/>
-<junction x="129.54" y="81.28"/>
-</segment>
-</net>
 <net name="N$14" class="0">
 <segment>
 <pinref part="J1" gate="G$1" pin="VBUS"/>
-<wire x1="20.32" y1="50.8" x2="27.94" y2="50.8" width="0.1524" layer="91"/>
-<pinref part="F1" gate="A" pin="1"/>
-<wire x1="27.94" y1="50.8" x2="27.94" y2="60.96" width="0.1524" layer="91"/>
+<wire x1="20.32" y1="50.8" x2="38.1" y2="50.8" width="0.1524" layer="91"/>
+<wire x1="38.1" y1="50.8" x2="38.1" y2="58.42" width="0.1524" layer="91"/>
+<pinref part="D4" gate="G$1" pin="A"/>
+<wire x1="38.1" y1="58.42" x2="33.02" y2="58.42" width="0.1524" layer="91"/>
 </segment>
 </net>
@@
 </segment>
 </net>
+<net name="N$16" class="0">
+<segment>
+<pinref part="S1" gate="G$1" pin="P"/>
+<wire x1="121.92" y1="83.82" x2="121.92" y2="81.28" width="0.1524" layer="91"/>
+<pinref part="R9" gate="G$1" pin="1"/>
+<pinref part="S1" gate="G$1" pin="P1"/>
+<wire x1="124.46" y1="78.74" x2="124.46" y2="81.28" width="0.1524" layer="91"/>
+<wire x1="124.46" y1="81.28" x2="124.46" y2="83.82" width="0.1524" layer="91"/>
+<wire x1="121.92" y1="81.28" x2="124.46" y2="81.28" width="0.1524" layer="91"/>
+<junction x="124.46" y="81.28"/>
+</segment>
+</net>
+<net name="N$11" class="0">
+<segment>
+<pinref part="D4" gate="G$1" pin="C"/>
+<wire x1="33.02" y1="63.5" x2="30.48" y2="63.5" width="0.1524" layer="91"/>
+<wire x1="30.48" y1="63.5" x2="30.48" y2="58.42" width="0.1524" layer="91"/>
+<wire x1="30.48" y1="58.42" x2="27.94" y2="58.42" width="0.1524" layer="91"/>
+<pinref part="F1" gate="A" pin="1"/>
+<wire x1="27.94" y1="58.42" x2="27.94" y2="60.96" width="0.1524" layer="91"/>
+</segment>
+</net>
